File: PCB/pcb_traversant/pcb_traversant.kicad_pcb (KiCad board)
At the start: 2 copper layers, 82 x 91.5 mm, 32 parts, among them J1 Conn_01x08_Pin, J2 Conn_01x02_Pin, J3 NEB_21_R, J4 Conn_01x01_Pin, U2 OPA2604AP, U3 OPA541AP

Commit message: Ajout plan de masse et via sur les 2 PCB
Connections:
- U3 pad 11: unconnected-(U3-Pad11) -> Net-(J4-Pin_1)
- U3 pad 4: unconnected-(U3-Pad4) -> Net-(C3-Pad2)
Routing:
- net Net-(J4-Pin_1): track 109.0 -> 114.8 mm
- net Net-(C3-Pad2): track 76.3 -> 82.1 mm
- net GND: vias 0 -> 9
- added copper zone on B.Cu, net GND
Other:
- board size 82 x 91.5 mm -> 81.8 x 91.5 mm
